File: Fascia_mainBoardV0/fasciaMainBoard_V0.brd (EAGLE design)
At the start: 61.5 x 40.6 mm, 168 parts, among them CN2 CA0612KRX7R9BB102, CN3 CA0612KRX7R9BB102, CN4 CA0612KRX7R9BB102, CN5 CA0612KRX7R9BB102, CN6 CA0612KRX7R9BB102, J1 0527450833, J2 MOLEX_52435-2271MOLEX_52435-2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, J3 -, J4 0527451633, J8 TC2030-MCP, Q1 BSS138PS,115, U1 ATSAMD21G-A, U10 ADUM5028, U11 TPD4E1B06DCKR, U12 TPD4E1B06DCKR, U13 TPD4E1B06DCKR, U14 TPD4E1B06DCKR, U15 TPD4E1B06DCKR, U16 TPD4E1B06DCKR, U17 MPU-6050, U18 LP5912Q3.3DRVRQ1, U2 ADS1299-X, U3 NINA-W102, U4 ATECC508A-MAHDA-T, U5 MCP73831T-4ADI_OT, U6 LM2664M6_NOPB, U7 TPS72325QDBVRQ1, U8 TLV70025DDCR, U9 LP5912Q3.3DRVRQ1, Y1 32.768Khz

Commit message: initial changes
Parts:
- removed C15: 10uF, SparkFun-Capacitors:0603
- removed C40, C42, C44, C47, C54, C56, C58, C60: 1uF, novaXR:0402-TIGHT
- removed C43, C45, C46, C55, C57, C59, C61, C66: 0.1uF, novaXR:0402-TIGHT
- removed C48: TAJA107K004RNJ, SamacSys_Parts:CAPPM3216X180N
- removed CLK, CS1, DRDY, MISO, MOSI, SCK: DNP, Arduino-utility:TP-0.8MM
- removed CN2, CN3, CN4, CN5, CN6: CA0612KRX7R9BB102, SamacSys_Parts:CA0612KRX7R9BB102
- removed FD4, FD5, FD6: DNP, Arduino-utility:FD-1-1.5
- removed J2: MOLEX_52435-2271MOLEX_52435-2271_0_0, Molex - 52435-2271:MOLEX_52435-2271_0
- removed J4: 0527451633, novaXR:0527451633
- removed J5: (no value), SparkFun-Connectors:JST-4-PTH
- removed J7: (no value), SparkFun-Connectors:1X03_SMD_RA_MALE
- removed R1, R30, R31, R32, R33: 10K, novaXR:0402-TIGHT
- removed R29: 1M, novaXR:0402-TIGHT
- removed RN1, RN2, RN3, RN4, RN5: CA0612KRX7R7BB104, SamacSys_Parts:CA0612KRX7R7BB104
- removed U11, U12, U13, U14, U15, U16: TPD4E1B06DCKR, SamacSys_Parts:SOT65P210X110-6N
- removed U2: ADS1299-X, SamacSys_Parts:QFP50P1200X1200X120-64N
- J1: value 0527450833 -> MOLEX_52435-2271MOLEX_52435-2271_0_0; device novaXR:0527450833 -> Molex - 52435-2271:MOLEX_52435-2271_0
- moved J1 18.3 mm to (46.3, 14.9), turned to 90 degrees
- moved C34 13.7 mm to (44.3, 23.1), turned to 90 degrees
- moved C36 12.1 mm to (43.5, 23.2)
- moved U17 8.21 mm to (33.7, 20.1), turned to 180 degrees
- moved R14 3.66 mm to (37.0, 17.2)
- moved PGND 3.01 mm to (50.0, 36.4)
- moved R9 1.96 mm to (31.1, 16.8)
- moved C53 1.30 mm to (39.8, 19.2)
- moved JTMS 0.92 mm to (33.4, 13.7)
- moved U4 0.85 mm to (39.0, 17.4)
- moved PB1 0.51 mm to (23.0, 20.5)
- moved C26 0.41 mm to (46.7, 28.3)
Connections:
- removed net 1N: J2.19, RN5.1, U14.4
- removed net 1P: J2.20, RN5.2, U15.1
- removed net 2N: J2.17, RN4.3, U14.2
- removed net 2P: J2.18, RN4.4, U14.5
- removed net 3N: J2.15, RN4.1, U13.4
- removed net 3P: J2.16, RN4.2, U14.1
- removed net 4N: J2.13, RN3.3, U13.2
- removed net 4P: J2.14, RN3.4, U13.5
- removed net 5N: J2.11, RN3.1, U12.4
- removed net 5P: J2.12, RN3.2, U13.1
- removed net 6N: J2.9, RN2.3, U12.2
- removed net 6P: J2.10, RN2.4, U12.5
- removed net 7N: J2.7, RN2.1, U11.4
- removed net 7P: J2.8, RN2.2, U12.1
- removed net 8N: J2.5, RN1.3, U11.2
- removed net 8P: J2.6, RN1.4, U11.5
- removed net ADS_CLK: CLK.X, J1.6, U2.37
- removed net BIAS: J2.4, RN1.2, U16.4
- removed net BIAS_DRV: C45.2, CN2.7, R29.2, RN1.6
- removed net BIAS_INV: J1.5, U2.61
- removed net IN1N: CN6.8, RN5.5, U2.15
- removed net IN1P: CN6.7, RN5.6, U2.16
- removed net IN2N: CN5.6, RN4.7, U2.13
- removed net IN2P: CN5.5, RN4.8, U2.14
- removed net IN3N: CN5.8, RN4.5, U2.11
- removed net IN3P: CN5.7, RN4.6, U2.12
- removed net IN4N: CN4.6, RN3.7, U2.9
- removed net IN4P: CN4.5, RN3.8, U2.10
- removed net IN5N: CN4.8, RN3.5, U2.7
- removed net IN5P: CN4.7, RN3.6, U2.8
- removed net IN6N: CN3.6, RN2.7, U2.5
- removed net IN6P: CN3.5, RN2.8, U2.6
- removed net IN7N: CN3.8, RN2.5, U2.3
- removed net IN7P: CN3.7, RN2.6, U2.4
- removed net IN8N: CN2.6, RN1.7, U2.1
- removed net IN8P: CN2.5, RN1.8, U2.2
- removed net N$22: C15.2, C66.1, U2.24
- removed net N$24: R33.2, U2.46
- removed net N$26: C45.1, R29.1, U2.62, U2.63
- removed net N$48: R32.2, U2.45
- removed net N$50: R31.2, U2.44
- removed net N$52: R30.2, U2.42
- removed net N$59: C40.1, U2.26
- removed net N$60: C48.1, U2.28
- removed net N$61: C42.1, U2.30
- removed net N$63: C46.2, C47.2, U2.55
- removed net N$66: R1.2, U2.38
- removed net SRB1: J5.3, RN5.3, U15.2
- removed net SRB2: J5.4, RN5.4, U15.5
- removed net _SRB1: CN6.6, RN5.7, U2.17
- removed net _SRB2: CN6.5, RN5.8, U2.18
- net ADS_RESET: now also J1.5; no longer U2.36
- net ADS_RESET2: no longer J4.5
- net AGND: now also J1.14, J1.15, J1.16; no longer C43.1, C44.1, CN2.1, CN2.2, CN2.3, CN2.4, CN2.8, CN3.1, CN3.2, CN3.3, CN3.4, CN4.1, CN4.2, CN4.3, CN4.4, CN5.1, CN5.2, CN5.3, CN5.4, CN6.1, CN6.2, CN6.3, CN6.4, J1.3, J1.4, J2.3, J5.2, R1.1, RN1.1, RN1.5, U11.3, U12.3, U13.3, U14.3, U15.3, U16.1, U16.3, U2.31, U2.41, U2.60
- net AVDD: now also J1.20, J1.21, J1.22; no longer C56.2, C57.2, C58.2, C59.2, C60.2, C61.2, J1.7, J1.8, J2.1, J2.2, U16.2, U2.19, U2.21, U2.22, U2.54, U2.56, U2.59
- net AVSS: now also J1.17, J1.18, J1.19; no longer C15.1, C40.2, C42.2, C43.2, C44.2, C46.1, C47.1, C48.2, C56.1, C57.1, C58.1, C59.1, C60.1, C61.1, C66.2, J1.1, J1.2, J2.21, J2.22, U15.4, U2.20, U2.23, U2.25, U2.32, U2.53, U2.57, U2.58
- net DVDD: now also J1.11, J1.12, J1.13; no longer C54.2, C55.2, J4.1, U2.35, U2.48, U2.50, U2.52
- net DVDD_ISO: no longer J4.11
- net GND: now also J1.10, J1.8, J1.9; no longer C54.1, C55.1, J4.10, J4.13, J4.15, R30.1, R31.1, R32.1, R33.1, U2.33, U2.49, U2.51
- net GND_ISO: no longer J4.12
- net PA02_EDA_SIG: now also J1.7; no longer J4.7
- net PA10_D2: no longer J7.2
- net PA16_S1_MOSI: now also J1.6; no longer J4.4, MOSI.X, U2.34
- net PA17_S1_SCK: now also J1.3; no longer J4.6, SCK.X, U2.40
- net PA19_S1_MISO: now also J1.2; no longer J4.14, MISO.X, U2.43
- net PA20_CS2: no longer J4.3
- net PA21_CS1: now also J1.4; no longer CS1.X, U2.39
- net PB02_DRDY2: no longer J4.2
- net PB03_A2: no longer J7.3
- net PB10_DRDY: now also J1.1; no longer DRDY.X, U2.47
- net RESET#: no longer J7.1
- net S0_I2C_SCL: no longer J4.8
- net S0_I2C_SDA: no longer J4.9
- net VCC: no longer J4.16
- net VDDANA: no longer J5.1
Routing:
- net VCC: track 143.2 -> 0.00 mm, vias 13 -> 0
- net GND: track 128.0 -> 0.00 mm, vias 27 -> 0
- net AVSS: track 118.0 -> 0.00 mm, vias 6 -> 0
- net AGND: track 93.5 -> 0.00 mm, vias 36 -> 0
- net AVDD: track 80.3 -> 0.00 mm, vias 7 -> 0
- net DVDD: track 74.0 -> 0.00 mm, vias 9 -> 0
- net PA30_SWCLK: track 67.9 -> 0.00 mm, vias 2 -> 0
- net PA31_SWDIO: track 62.4 -> 0.00 mm, vias 4 -> 0
- net PA28_ACK: track 53.0 -> 0.00 mm, vias 4 -> 0
- net PA17_S1_SCK: track 52.0 -> 0.00 mm, vias 3 -> 0
- net PA19_S1_MISO: track 48.0 -> 0.00 mm, vias 4 -> 0
- net PA16_S1_MOSI: track 42.5 -> 0.00 mm, vias 3 -> 0
- net PA27_GPIO0: track 41.1 -> 0.00 mm, vias 3 -> 0
- net PA20_CS2: track 40.1 -> 0.00 mm, vias 3 -> 0
- net GND_ISO: track 36.7 -> 0.00 mm, vias 5 -> 0
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- removed copper zone on layer 15, net AGND
- removed copper zone on layer 16, net AGND
- removed copper zone on layer 16, net AVDD
- removed copper zone on layer 2, net AVDD
- removed copper zone on layer 16, net AVSS
- removed copper zone on layer 2, net AVSS
Other:
- board size 61.5 x 40.6 mm -> 33.6 x 40.6 mm
- board text removed: "NOVAXR_mainBoard_V2 _10/10/2019"
- board text removed: "SRB1"
- board text removed: "SRB2"
- board text removed: "VDDANA"

Commit message: added files for the physioBoard
Routing:
- removed copper zone on layer 1, net AGND
- removed copper zone on layer 1, net AVSS
- removed copper zone on layer 2, net DVDD
- removed copper zone on layer 1, net GND
- removed copper zone on layer 15, net GND
- removed copper zone on layer 16, net GND
- removed copper zone on layer 16, net GND_ISO

Commit message: minor updates
Parts:
- removed C41, C64: 10uF, SparkFun-Capacitors:0603
- removed C49: 0.1uF, novaXR:0402-TIGHT
- removed C51: 0.22uF, novaXR:0402-TIGHT
- removed L1, L2: BLM15HD182SN1D, SamacSys_Parts:INDC1005X55N
- removed U10: ADUM5028, novaXR:SOIC_IC
- J1: value MOLEX_52435-2271MOLEX_52435-2271_0_0 -> MOLEX_52437-2471MOLEX_52437-2471_0_0; device Molex - 52435-2271:MOLEX_52435-2271_0 -> Molex - 52437-2471:MOLEX_52437-2471_0
- moved FD1 49.6 mm to (35.8, 52.5), turned to 180 degrees
- moved FD3 46.0 mm to (35.8, 51.0), turned to 180 degrees
- moved D3 45.2 mm to (53.1, 44.6), turned to 90 degrees
- moved JGND 43.2 mm to (38.4, 52.4), turned to 270 degrees
- moved R13 42.6 mm to (37.4, 49.0), turned to 90 degrees
- moved R17 41.9 mm to (54.2, 41.2), turned to 270 degrees
- moved C13 41.4 mm to (39.2, 48.4), turned to 180 degrees
- moved U3 40.9 mm to (45.3, 46.8), turned to 90 degrees
- moved R16 40.2 mm to (53.1, 41.1), turned to 270 degrees
- moved RST 40.1 mm to (48.5, 46.7), turned to 180 degrees
- moved C12 39.4 mm to (39.2, 47.4), turned to 0 degrees
- moved R15 38.6 mm to (52.0, 41.1), turned to 270 degrees
- moved R4 37.6 mm to (37.4, 46.5), turned to 270 degrees
- moved JCLK 36.1 mm to (47.3, 43.4), turned to 270 degrees
- moved C28 35.9 mm to (39.2, 45.6), turned to 180 degrees
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Connections:
- new net ADS_CLK: J1.24
- new net BIAS_INV: J1.1
- new net N$14: J1.11
- new net N$22: J1.3
- new net N$24: J1.6
- new net N$26: J1.9
- new net PA07_DRDY2: J1.23
- net ADS_RESET: no longer J1.5
- net ADS_RESET2: now also J1.20
- net AGND: now also J1.8; no longer J1.14, J1.15, J1.16
- net AVDD: now also J1.4; no longer J1.20, J1.21, J1.22
- net AVSS: now also J1.5; no longer J1.17, J1.18, J1.19
- net DVDD: now also J1.10; no longer C41.2, C49.2, J1.11, J1.12, J1.13, U10.3
- net DVDD_ISO: no longer C64.2, L1.2
- net GND: now also J1.13, J1.14, J1.15; no longer C41.1, C49.1, J1.10, J1.8, J1.9, U10.1, U10.2, U10.4
- net GND_ISO: no longer C51.1, C64.1, L2.1, L2.2, U10.5, U10.7, U10.8
- net N$5: now also J1.7; no longer C51.2, L1.1, U10.6
- net PA02_EDA_SIG: now also J1.2; no longer J1.7
- net PA16_S1_MOSI: now also J1.21; no longer J1.6
- net PA17_S1_SCK: now also J1.19; no longer J1.3
- net PA19_S1_MISO: now also J1.18; no longer J1.2
- net PA20_CS2: now also J1.22
- net PA21_CS1: no longer J1.4
- net PB10_DRDY: no longer J1.1
- net S0_I2C_SCL: now also J1.16
- net S0_I2C_SDA: now also J1.17
- net VCC: now also J1.12
Routing:
- net PB08_RST: track 1.59 -> 0.00 mm
Other:
- outline, holes or cut-outs redrawn

Commit message: MINOR CHANGES
Parts:
- moved Q1 13.3 mm to (48.2, 35.8), turned to 0 degrees
- moved C35 10.5 mm to (45.0, 38.8), turned to 270 degrees
- moved R18 6.90 mm to (40.7, 38.8)
- moved C37 6.17 mm to (43.0, 38.8), turned to 270 degrees
- moved C36 4.83 mm to (38.4, 34.5)
- moved C34 4.76 mm to (37.4, 34.5)
- moved R7 3.29 mm to (40.6, 38.8), turned to 90 degrees
- moved R11 2.80 mm to (50.6, 35.1), turned to 90 degrees
- moved C23 2.44 mm to (27.9, 23.3), turned to 90 degrees
- moved R14 2.38 mm to (41.6, 38.8)
- moved R9 2.34 mm to (46.0, 36.4)
- moved R10 2.21 mm to (50.6, 37.3), turned to 270 degrees
- moved R20 1.90 mm to (41.4, 30.1)
- moved R12 1.49 mm to (48.7, 37.5)
- moved TX 1.17 mm to (56.3, 24.6)
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Connections:
- net PB02_DRDY2 renamed PB02_DRDY
- removed net ADS_RESET2: J1.20, U1.31
- removed net BIAS_INV: J1.1
- removed net N$14: J1.11
- removed net N$22: J1.3
- removed net N$24: J1.6
- removed net N$26: J1.9
- removed net N$5: J1.7
- removed net PA07_DRDY2: J1.23
- removed net PA20_CS2: J1.22, U1.29
- removed net PB10_DRDY: U1.19
- new net PA07_DRDY: J1.18
- new net PA20_CS: J1.21, U1.29
- net ADS_CLK: now also J1.22; no longer J1.24
- net ADS_RESET: now also J1.23
- net AGND: now also J1.7
- net AVDD: now also J1.3
- net AVSS: now also J1.6
- net DVDD: now also J1.9
- net PA16_S1_MOSI: now also J1.24; no longer J1.21
- net PA17_S1_SCK: now also J1.20; no longer J1.19
- net PA19_S1_MISO: now also J1.19; no longer J1.18
- net VCC: now also J1.11
Routing:
- net AVSS: track 0.00 -> 6.36 mm, vias 0 -> 2
- net AVDD: track 0.00 -> 5.19 mm, vias 0 -> 2
- net PA02_EDA_SIG: track 0.00 -> 2.22 mm
- added copper zone on layer 2, net AGND
- added copper zone on layer 16, net AVDD
- added copper zone on layer 15, net AVSS
- added copper zone on layer 2, net GND

Commit message: MINOR CHANGES
Parts:
- moved C34 8.30 mm to (35.8, 42.6), turned to 180 degrees
- moved C36 7.56 mm to (35.8, 41.6), turned to 180 degrees
- moved U17 6.05 mm to (36.8, 37.6), turned to 270 degrees
- moved D4 0.32 mm to (44.1, 30.6)
- moved D5 0.32 mm to (44.1, 31.6)
- moved D2 0.10 mm to (49.0, 30.9)
Connections:
- removed net PB02_DRDY: U1.47
- net PA07_DRDY: now also U1.12
Routing:
- net PA17_S1_SCK: track 0.00 -> 19.2 mm, vias 0 -> 1
- net ADS_RESET: track 0.00 -> 18.5 mm, vias 0 -> 1
- net PA19_S1_MISO: track 0.00 -> 18.4 mm, vias 0 -> 1
- net PA16_S1_MOSI: track 0.00 -> 18.2 mm, vias 0 -> 1
- net PA20_CS: track 0.00 -> 18.1 mm, vias 0 -> 1
- net PA07_DRDY: track 0.00 -> 9.58 mm, vias 0 -> 1
- added copper zone on layer 15, net VCC

Commit message: Update fasciaMainBoard_V0.brd
Parts:
- moved C35 9.43 mm to (36.3, 35.0), turned to 0 degrees
- moved C37 3.81 mm to (39.7, 37.1), turned to 90 degrees
- moved R7 3.59 mm to (39.8, 35.3), turned to 0 degrees
- moved R18 3.47 mm to (40.8, 35.3), turned to 180 degrees
- moved U17 0.81 mm to (36.7, 38.4)
- moved R14 0.70 mm to (41.6, 38.1)
- moved R8 0.70 mm to (41.6, 38.1)
- moved C53 0.32 mm to (36.4, 36.5)
Routing:
- net S0_I2C_SDA: track 0.00 -> 17.5 mm, vias 0 -> 1
- net S0_I2C_SCL: track 0.00 -> 6.78 mm, vias 0 -> 1
- net N$37: track 0.00 -> 1.44 mm
- net N$39: track 0.00 -> 1.03 mm

Commit message: progress on routing
Parts:
- moved R11 8.22 mm to (44.2, 40.4), turned to 270 degrees
- moved R10 7.93 mm to (43.3, 40.4)
- moved FD1 7.02 mm to (29.9, 48.7)
- moved R12 6.87 mm to (42.4, 40.3), turned to 270 degrees
- moved FD3 6.33 mm to (29.9, 48.7)
- moved PGND 5.83 mm to (30.8, 22.7)
- moved Q1 5.12 mm to (43.2, 36.7), turned to 90 degrees
- moved C16 4.07 mm to (49.0, 28.4), turned to 0 degrees
- moved GPIO0 3.18 mm to (47.2, 39.3)
- moved D+1 2.94 mm to (47.1, 32.1)
- moved R9 2.93 mm to (43.7, 34.6), turned to 180 degrees
- moved D-1 2.82 mm to (47.2, 30.1)
- moved JGND 2.62 mm to (38.7, 49.8)
- moved R21 2.42 mm to (41.7, 28.6)
- moved R14 2.40 mm to (41.6, 40.5)
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Connections:
- removed net PB03_A2: U1.48
- new net MPU_INT: U1.48, U17.12
- net VBAT_LVL: now also U1.47; no longer U1.10
Routing:
- net GND: track 0.00 -> 136.2 mm, vias 0 -> 30
- net VCC: track 0.00 -> 56.3 mm, vias 0 -> 14
- net PA31_SWDIO: track 0.00 -> 50.9 mm, vias 0 -> 2
- net AGND: track 0.00 -> 48.5 mm, vias 0 -> 6
- net PB23_S5_RX: track 0.00 -> 41.4 mm, vias 0 -> 3
- net PA30_SWCLK: track 0.00 -> 39.1 mm, vias 0 -> 3
- net DVDD: track 0.00 -> 36.2 mm
- net PA28_ACK: track 0.00 -> 35.0 mm, vias 0 -> 2
- net PB22_S5_TX: track 0.00 -> 34.7 mm, vias 0 -> 2
- net N$12: track 0.00 -> 33.1 mm, vias 0 -> 3
- net N$21: track 0.00 -> 30.0 mm, vias 0 -> 1
- net PA02_EDA_SIG: track 2.22 -> 26.2 mm, vias 0 -> 1
- net N$40: track 0.00 -> 23.0 mm
- net V_BATT: track 0.00 -> 22.2 mm, vias 0 -> 1
- net _V_BATT: track 0.00 -> 21.2 mm, vias 0 -> 1
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- added copper zone on layer 1, net GND

Commit message: maiboard routing completed
Parts:
- added CS, MISO, MOSI, SCK: DNP, Arduino-utility:TP-0.8MM
- added FD4, FD5, FD6: DNP, Arduino-utility:FD-1-1.5
- moved FD2 16.9 mm to (45.3, 16.7)
- moved FD3 5.80 mm to (34.1, 44.7)
- moved RST 1.00 mm to (49.5, 46.7)
- moved C22 0.61 mm to (27.6, 19.7)
- moved C28 0.20 mm to (39.2, 45.8)
- moved R10 0.20 mm to (43.5, 40.4)
- moved R12 0.20 mm to (42.6, 40.3)
- moved R14 0.14 mm to (41.7, 40.4)
- moved R11 0.10 mm to (44.3, 40.4)
Connections:
- net PA16_S1_MOSI: now also MOSI.X
- net PA17_S1_SCK: now also SCK.X
- net PA19_S1_MISO: now also MISO.X
- net PA20_CS: now also CS.X
Routing:
- net DVDD: track 36.2 -> 58.4 mm
- net AGND: track 48.5 -> 39.1 mm, vias 6 -> 7
- net PA19_S1_MISO: track 19.1 -> 22.5 mm, vias 1 -> 2
- net PA17_S1_SCK: track 19.3 -> 21.9 mm, vias 1 -> 2
- net GND: track 136.2 -> 138.9 mm, vias 30 -> 33
- net PA20_CS: track 18.5 -> 20.7 mm, vias 1 -> 2
- net PA16_S1_MOSI: track 18.9 -> 21.1 mm, vias 1 -> 2
- net VCC: track 56.3 -> 57.9 mm, vias 14 -> 15
- net N$12: track 33.1 -> 34.2 mm
- net -RAW: track 11.2 -> 10.2 mm
- net PA28_ACK: track 35.0 -> 34.4 mm
Other:
- board text added: "CS"
- board text added: "FACIA_MAINBOARD_V0_11/21/19"
- board text removed: "A2"
- board text removed: "D+1"
- board text removed: "D-1"
- board text removed: "D2"
- board text removed: "RESET#"
