File: Fascia_mainBoardV0/fasciaMainBoard_V0.brd (EAGLE design)
At the start: 33.6 x 40.6 mm, 114 parts, among them J1 MOLEX_52437-2471MOLEX_52437-2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, J3 -, J8 TC2030-MCP, Q1 BSS138PS,115, U1 ATSAMD21G-A, U17 MPU-6050, U18 LP5912Q3.3DRVRQ1, U3 NINA-W102, U4 ATECC508A-MAHDA-T, U5 MCP73831T-4ADI_OT, U6 LM2664M6_NOPB, U7 TPS72325QDBVRQ1, U8 TLV70025DDCR, U9 LP5912Q3.3DRVRQ1, Y1 32.768Khz

Commit message: files ready for manufacture
Changed lines of the file:
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@@
 <?xml version="1.0" encoding="utf-8"?>
 <!DOCTYPE eagle SYSTEM "eagle.dtd">
-<eagle version="9.5.1">
+<eagle version="9.5.2">
 <drawing>
 <settings>
@@
 <layer number="19" name="Unrouted" color="6" fill="1" visible="yes" active="yes"/>
 <layer number="20" name="Dimension" color="24" fill="1" visible="yes" active="yes"/>
-<layer number="21" name="tPlace" color="7" fill="1" visible="no" active="yes"/>
+<layer number="21" name="tPlace" color="7" fill="1" visible="yes" active="yes"/>
 <layer number="22" name="bPlace" color="7" fill="1" visible="yes" active="yes"/>
 <layer number="23" name="tOrigins" color="15" fill="1" visible="yes" active="yes"/>
@@
 <text x="27.2" y="32.5" size="0.6096" layer="26" ratio="20" rot="MR180">MOSI</text>
 <text x="28.3" y="33.9" size="0.6096" layer="26" ratio="20" rot="MR180">CS</text>
-<text x="31.6" y="51.7" size="0.8128" layer="25" ratio="13" distance="61">FACIA_MAINBOARD_V0_11/21/19</text>
+<text x="30.9" y="52.1" size="0.8128" layer="25" ratio="13" distance="61">FACIA_MAINBOARD_V0_11/21/19</text>
 </plain>
 <attributes>
@@
 <contactref element="RST" pad="X"/>
 <contactref element="U3" pad="19"/>
-<wire x1="49.711" y1="46.627" x2="48.727" y2="46.627" width="0.254" layer="16"/>
-<wire x1="48.727" y1="46.627" x2="48.7" y2="46.6" width="0.254" layer="16"/>
-<wire x1="48.7" y1="46.6" x2="48.566765625" y2="46.6" width="0.254" layer="16"/>
-<wire x1="48.566765625" y1="46.6" x2="48.476" y2="46.690765625" width="0.254" layer="16"/>
 <via x="48.476" y="46.690765625" extent="1-16" drill="0.25"/>
 <wire x1="42.605796875" y1="39.839090625" x2="42.559" y2="39.79229375" width="0.3048" layer="1"/>
@@
 <via x="35.8" y="45.2" extent="1-16" drill="0.25"/>
 <wire x1="35.8" y1="45.2" x2="35.8" y2="46.1" width="0.3048" layer="1"/>
-<wire x1="47.609234375" y1="46.690765625" x2="49.476" y2="46.690765625" width="0.3048" layer="1"/>
 <wire x1="38.0806" y1="44.700925" x2="37.779675" y2="44.4" width="0.3048" layer="16"/>
 <wire x1="35.7" y1="44.7" x2="35.7" y2="45.1" width="0.3048" layer="16"/>
 <wire x1="35.8" y1="46.1" x2="37.4" y2="47.7" width="0.3048" layer="1"/>
 <wire x1="37.4" y1="47.7" x2="46.6" y2="47.7" width="0.3048" layer="1"/>
-<wire x1="46.6" y1="47.7" x2="47.609234375" y2="46.690765625" width="0.3048" layer="1"/>
-<wire x1="49.476" y1="46.690765625" x2="49.711" y2="46.627" width="0" layer="19" extent="1-16"/>
+<wire x1="47.609234375" y1="46.690765625" x2="46.6" y2="47.7" width="0.3048" layer="1"/>
+<wire x1="49.711" y1="46.627" x2="49.647234375" y2="46.690765625" width="0.3048" layer="16"/>
+<wire x1="49.647234375" y1="46.690765625" x2="48.476" y2="46.690765625" width="0.3048" layer="16"/>
+<wire x1="48.476" y1="46.690765625" x2="49.476" y2="46.690765625" width="0.3048" layer="1"/>
+<wire x1="48.476" y1="46.690765625" x2="47.609234375" y2="46.690765625" width="0.3048" layer="1"/>
 </signal>
 <signal name="N$11">
