File: Fascia_mainBoardV0/fasciaMainBoard_V0.sch (EAGLE design)
At the start: 168 parts, among them CN2 CA0612KRX7R9BB102, CN3 CA0612KRX7R9BB102, CN4 CA0612KRX7R9BB102, CN5 CA0612KRX7R9BB102, CN6 CA0612KRX7R9BB102, J1 0527450833, J2 MOLEX_52435-2271MOLEX_52435-2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, J3 -, J4 0527451633, J8 TC2030-MCP, Q1 BSS138PS,115, U1 ATSAMD21G-A, U10 ADUM5028, U11 TPD4E1B06DCKR, U12 TPD4E1B06DCKR, U13 TPD4E1B06DCKR, U14 TPD4E1B06DCKR, U15 TPD4E1B06DCKR, U16 TPD4E1B06DCKR, U17 MPU-6050, U18 LP5912Q3.3DRVRQ1, U2 ADS1299-X, U3 NINA-W102, U4 ATECC508A-MAHDA-T, U5 MCP73831T-4ADI_OT, U6 LM2664M6_NOPB, U7 TPS72325QDBVRQ1, U8 TLV70025DDCR, U9 LP5912Q3.3DRVRQ1, Y1 32.768Khz

Commit message: initial changes
Parts:
- removed C15: 10uF, SparkFun-Capacitors:10UF-0603-6.3V-20%
- removed C40, C42, C44, C47, C54, C56, C58, C60: 1uF, novaXR:1UF-0402T-16V-10%
- removed C43, C45, C46, C55, C57, C59, C61, C66: 0.1uF, novaXR:0.1UF-0402T-16V-10%
- removed C48: TAJA107K004RNJ, SamacSys_Parts:TAJA107K004RNJ
- removed CLK, CS1, DRDY, MISO, MOSI, SCK: DNP, Arduino-utility:TPTP-0.8MM
- removed CN2, CN3, CN4, CN5, CN6: CA0612KRX7R9BB102, SamacSys_Parts:CA0612KRX7R9BB102
- removed FD4, FD5, FD6: DNP, Arduino-utility:FIDUCIAL-1.5MM
- removed J2: MOLEX_52435-2271MOLEX_52435-2271_0_0, Molex - 52435-2271:MOLEX_52435-2271MOLEX_52435-2271_0_0
- removed J4: 0527451633, novaXR:0527451633
- removed J5: (no value), SparkFun-Connectors:CONN_04JST-PTH
- removed J7: (no value), SparkFun-Connectors:CONN_03SMD_RA_MALE
- removed R1, R30, R31, R32, R33: 10K, novaXR:10K
- removed R29: 1M, novaXR:1M
- removed RN1, RN2, RN3, RN4, RN5: CA0612KRX7R7BB104, SamacSys_Parts:CA0612KRX7R7BB104
- removed U11, U12, U13, U14, U15, U16: TPD4E1B06DCKR, SamacSys_Parts:TPD4E1B06DCKR
- removed U2: ADS1299-X, SamacSys_Parts:ADS1299-X
- J1: value 0527450833 -> MOLEX_52435-2271MOLEX_52435-2271_0_0; device novaXR:0527450833 -> Molex - 52435-2271:MOLEX_52435-2271MOLEX_52435-2271_0_0
Connections:
- removed net 1N: J2.19, RN5.P$1, U14.IO3
- removed net 1P: J2.20, RN5.P$2, U15.IO1
- removed net 2N: J2.17, RN4.P$3, U14.IO2
- removed net 2P: J2.18, RN4.P$4, U14.IO4
- removed net 3N: J2.15, RN4.P$1, U13.IO3
- removed net 3P: J2.16, RN4.P$2, U14.IO1
- removed net 4N: J2.13, RN3.P$3, U13.IO2
- removed net 4P: J2.14, RN3.P$4, U13.IO4
- removed net 5N: J2.11, RN3.P$1, U12.IO3
- removed net 5P: J2.12, RN3.P$2, U13.IO1
- removed net 6N: J2.9, RN2.P$3, U12.IO2
- removed net 6P: J2.10, RN2.P$4, U12.IO4
- removed net 7N: J2.7, RN2.P$1, U11.IO3
- removed net 7P: J2.8, RN2.P$2, U12.IO1
- removed net 8N: J2.5, RN1.P$3, U11.IO2
- removed net 8P: J2.6, RN1.P$4, U11.IO4
- removed net ADS_CLK: CLK.P$1, J1.6, U2.CLK
- removed net BIAS: J2.4, RN1.P$2, U16.IO3
- removed net BIAS_DRV: C45.2, CN2.C16, R29.2, RN1.P$6
- removed net BIAS_INV: J1.5, U2.BIASINV
- removed net IN1N: CN6.C17, RN5.P$5, U2.IN1N
- removed net IN1P: CN6.C16, RN5.P$6, U2.IN1P
- removed net IN2N: CN5.C15, RN4.P$7, U2.IN2N
- removed net IN2P: CN5.C14, RN4.P$8, U2.IN2P
- removed net IN3N: CN5.C17, RN4.P$5, U2.IN3N
- removed net IN3P: CN5.C16, RN4.P$6, U2.IN3P
- removed net IN4N: CN4.C15, RN3.P$7, U2.IN4N
- removed net IN4P: CN4.C14, RN3.P$8, U2.IN4P
- removed net IN5N: CN4.C17, RN3.P$5, U2.IN5N
- removed net IN5P: CN4.C16, RN3.P$6, U2.IN5P
- removed net IN6N: CN3.C15, RN2.P$7, U2.IN6N
- removed net IN6P: CN3.C14, RN2.P$8, U2.IN6P
- removed net IN7N: CN3.C17, RN2.P$5, U2.IN7N
- removed net IN7P: CN3.C16, RN2.P$6, U2.IN7P
- removed net IN8N: CN2.C15, RN1.P$7, U2.IN8N
- removed net IN8P: CN2.C14, RN1.P$8, U2.IN8P
- removed net N$22: C15.2, C66.1, U2.VREFP
- removed net N$24: R33.2, U2.GPIO4
- removed net N$26: C45.1, R29.1, U2.BIASIN, U2.BIASOUT
- removed net N$48: R32.2, U2.GPIO3
- removed net N$50: R31.2, U2.GPIO2
- removed net N$52: R30.2, U2.GPIO1
- removed net N$59: C40.1, U2.VCAP4
- removed net N$60: C48.+, U2.VCAP1
- removed net N$61: C42.1, U2.VCAP2
- removed net N$63: C46.2, C47.2, U2.VCAP3
- removed net N$66: R1.2, U2.START
- removed net SRB1: J5.3, RN5.P$3, U15.IO2
- removed net SRB2: J5.4, RN5.P$4, U15.IO4
- removed net _SRB1: CN6.C15, RN5.P$7, U2.SRB1
- removed net _SRB2: CN6.C14, RN5.P$8, U2.SRB2
- net ADS_RESET: now also J1.5; no longer U2.!RESET
- net ADS_RESET2: no longer J4.5
- net AGND: now also J1.14, J1.15, J1.16; no longer C43.1, C44.1, CN2.C10, CN2.C11, CN2.C12, CN2.C13, CN2.C17, CN3.C10, CN3.C11, CN3.C12, CN3.C13, CN4.C10, CN4.C11, CN4.C12, CN4.C13, CN5.C10, CN5.C11, CN5.C12, CN5.C13, CN6.C10, CN6.C11, CN6.C12, CN6.C13, J1.3, J1.4, J2.3, J5.2, R1.1, RN1.P$1, RN1.P$5, U11.GND, U12.GND, U13.GND, U14.GND, U15.GND, U16.GND, U16.IO1, U2.BIASREF, U2.DAISY_IN, U2.RESV1
- net AVDD: now also J1.20, J1.21, J1.22; no longer C56.2, C57.2, C58.2, C59.2, C60.2, C61.2, J1.7, J1.8, J2.1, J2.2, U16.IO2, U2.AVDD1, U2.AVDD_1, U2.AVDD_2, U2.AVDD_3, U2.AVDD_4, U2.AVDD_5
- net AVSS: now also J1.17, J1.18, J1.19; no longer C15.1, C40.2, C42.2, C43.2, C44.2, C46.1, C47.1, C48.-, C56.1, C57.1, C58.1, C59.1, C60.1, C61.1, C66.2, J1.1, J1.2, J2.21, J2.22, U15.IO3, U2.AVSS1, U2.AVSS_1, U2.AVSS_2, U2.AVSS_3, U2.AVSS_4, U2.AVSS_5, U2.VREFN
- net DVDD: now also J1.11, J1.12, J1.13; no longer C54.2, C55.2, J4.1, U2.!PWDN, U2.CLKSEL, U2.DVDD_1, U2.DVDD_2
- net DVDD_ISO: no longer J4.11
- net GND: now also J1.10, J1.8, J1.9; no longer C54.1, C55.1, J4.10, J4.13, J4.15, R30.1, R31.1, R32.1, R33.1, U2.DGND_1, U2.DGND_2, U2.DGND_3
- net GND_ISO: no longer J4.12
- net PA02_EDA_SIG: now also J1.7; no longer J4.7
- net PA10_D2: no longer J7.2
- net PA16_S1_MOSI: now also J1.6; no longer J4.4, MOSI.P$1, U2.DIN
- net PA17_S1_SCK: now also J1.3; no longer J4.6, SCK.P$1, U2.SCLK
- net PA19_S1_MISO: now also J1.2; no longer J4.14, MISO.P$1, U2.DOUT
- net PA20_CS2: no longer J4.3
- net PA21_CS1: now also J1.4; no longer CS1.P$1, U2.!CS
- net PB02_DRDY2: no longer J4.2
- net PB03_A2: no longer J7.3
- net PB10_DRDY: now also J1.1; no longer DRDY.P$1, U2.!DRDY
- net RESET#: no longer J7.1
- net S0_I2C_SCL: no longer J4.8
- net S0_I2C_SDA: no longer J4.9
- net VCC: no longer J4.16
- net VDDANA: no longer J5.1
Other:
- note removed: "2.2K"
- note removed: "Following latest version MFG Januiary 2017 for the ADS1299 http://www.ti.com/lit/ds/symlink/ads1299.pdf"
- note removed: "openBCI"

Commit message: minor updates
Parts:
- removed C41, C64: 10uF, SparkFun-Capacitors:10UF-0603-6.3V-20%
- removed C49: 0.1uF, novaXR:0.1UF-0402T-16V-10%
- removed C51: 0.22uF, novaXR:0.22UF-0402T-16V-10%
- removed L1, L2: BLM15HD182SN1D, SamacSys_Parts:BLM15HD182SN1D
- removed U10: ADUM5028, novaXR:ADUM5028
- J1: value MOLEX_52435-2271MOLEX_52435-2271_0_0 -> MOLEX_52437-2471MOLEX_52437-2471_0_0; device Molex - 52435-2271:MOLEX_52435-2271MOLEX_52435-2271_0_0 -> Molex - 52437-2471:MOLEX_52437-2471MOLEX_52437-2471_0_0
Connections:
- new net ADS_CLK: J1.24
- new net BIAS_INV: J1.1
- new net N$14: J1.11
- new net N$22: J1.3
- new net N$24: J1.6
- new net N$26: J1.9
- new net PA07_DRDY2: J1.23
- net ADS_RESET: no longer J1.5
- net ADS_RESET2: now also J1.20
- net AGND: now also J1.8; no longer J1.14, J1.15, J1.16
- net AVDD: now also J1.4; no longer J1.20, J1.21, J1.22
- net AVSS: now also J1.5; no longer J1.17, J1.18, J1.19
- net DVDD: now also J1.10; no longer C41.2, C49.2, J1.11, J1.12, J1.13, U10.VDDP
- net DVDD_ISO: no longer C64.2, L1.2
- net GND: now also J1.13, J1.14, J1.15; no longer C41.1, C49.1, J1.10, J1.8, J1.9, U10.GND, U10.GND1, U10.PDIS
- net GND_ISO: no longer C51.1, C64.1, L2.1, L2.2, U10.GND-ISO, U10.GND-ISO1, U10.VSEL
- net N$5: now also J1.7; no longer C51.2, L1.1, U10.VISO
- net PA02_EDA_SIG: now also J1.2; no longer J1.7
- net PA16_S1_MOSI: now also J1.21; no longer J1.6
- net PA17_S1_SCK: now also J1.19; no longer J1.3
- net PA19_S1_MISO: now also J1.18; no longer J1.2
- net PA20_CS2: now also J1.22
- net PA21_CS1: no longer J1.4
- net PB10_DRDY: no longer J1.1
- net S0_I2C_SCL: now also J1.16
- net S0_I2C_SDA: now also J1.17
- net VCC: now also J1.12
Other:
- note removed: "ADUM5028"

Commit message: MINOR CHANGES
Connections:
- net PB02_DRDY2 renamed PB02_DRDY
- removed net ADS_RESET2: J1.20, U1.PA22(I2C/SER3:0+)
- removed net BIAS_INV: J1.1
- removed net N$14: J1.11
- removed net N$22: J1.3
- removed net N$24: J1.6
- removed net N$26: J1.9
- removed net N$5: J1.7
- removed net PA07_DRDY2: J1.23
- removed net PA20_CS2: J1.22, U1.PA20(SER5:2+)
- removed net PB10_DRDY: U1.PB10(SER4:2+)
- new net PA07_DRDY: J1.18
- new net PA20_CS: J1.21, U1.PA20(SER5:2+)
- net ADS_CLK: now also J1.22; no longer J1.24
- net ADS_RESET: now also J1.23
- net AGND: now also J1.7
- net AVDD: now also J1.3
- net AVSS: now also J1.6
- net DVDD: now also J1.9
- net PA16_S1_MOSI: now also J1.24; no longer J1.21
- net PA17_S1_SCK: now also J1.20; no longer J1.19
- net PA19_S1_MISO: now also J1.19; no longer J1.18
- net VCC: now also J1.11

Commit message: MINOR CHANGES
Connections:
- removed net PB02_DRDY: U1.PB02(AIN10/SER5:0)
- net PA07_DRDY: now also U1.PA07(AIN7/SER0:3/TC1:1)
Changed lines of the file:
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@@
-</segment>
-</net>
-<net name="PB02_DRDY" class="0">
-<segment>
-<pinref part="U1" gate="G$1" pin="PB02(AIN10/SER5:0)"/>
-<wire x1="276.86" y1="200.66" x2="266.7" y2="200.66" width="0.1524" layer="91"/>
-<label x="266.7" y="200.66" size="1.016" layer="95" rot="R180" xref="yes"/>
 </segment>
 </net>
@@
 </segment>
 </net>
-<net name="PA07_DRDY" class="0">
-<segment>
-<label x="287.02" y="58.42" size="1.016" layer="95" rot="R180" xref="yes"/>
-<wire x1="299.5676" y1="58.42" x2="297.18" y2="58.42" width="0.1524" layer="91"/>
-<pinref part="J1" gate="G$0" pin="18"/>
-<wire x1="297.18" y1="58.42" x2="287.02" y2="58.42" width="0.1524" layer="91"/>
-<wire x1="299.5676" y1="58.42" x2="302.006" y2="58.42" width="0.1524" layer="91"/>
-</segment>
-</net>
 <net name="PA20_CS" class="0">
 <segment>
@@
 </segment>
 </net>
+<net name="PA07_DRDY" class="0">
+<segment>
+<pinref part="U1" gate="G$1" pin="PA07(AIN7/SER0:3/TC1:1)"/>
+<wire x1="276.86" y1="203.2" x2="266.7" y2="203.2" width="0.1524" layer="91"/>
+<label x="266.7" y="203.2" size="1.016" layer="95" rot="R180" xref="yes"/>
+</segment>
+<segment>
+<label x="287.02" y="58.42" size="1.016" layer="95" rot="R180" xref="yes"/>
+<wire x1="299.5676" y1="58.42" x2="297.18" y2="58.42" width="0.1524" layer="91"/>
+<pinref part="J1" gate="G$0" pin="18"/>
+<wire x1="297.18" y1="58.42" x2="287.02" y2="58.42" width="0.1524" layer="91"/>
+<wire x1="299.5676" y1="58.42" x2="302.006" y2="58.42" width="0.1524" layer="91"/>
+</segment>
+</net>

Commit message: progress on routing
Connections:
- removed net PB03_A2: U1.PB03(AIN11/SER5:1)
- new net MPU_INT: U1.PB03(AIN11/SER5:1), U17.INT
- net VBAT_LVL: now also U1.PB02(AIN10/SER5:0); no longer U1.PA05(AIN5/SER0:1/TC0:1)
Changed lines of the file:
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@@
 <setting verticaltext="up"/>
 </settings>
-<grid distance="0.1" unitdist="inch" unit="inch" style="dots" multiple="1" display="yes" altdistance="0.01" altunitdist="inch" altunit="inch"/>
+<grid distance="0.1" unitdist="inch" unit="inch" style="lines" multiple="1" display="no" altdistance="0.01" altunitdist="inch" altunit="inch"/>
 <layers>
 <layer number="1" name="Top" color="4" fill="1" visible="no" active="no"/>
@@
 <net name="VBAT_LVL" class="0">
 <segment>
-<pinref part="U1" gate="G$1" pin="PA05(AIN5/SER0:1/TC0:1)"/>
-<wire x1="276.86" y1="208.28" x2="264.16" y2="208.28" width="0.1524" layer="91"/>
-<label x="264.16" y="208.28" size="1.016" layer="95" rot="R180" xref="yes"/>
+<pinref part="U1" gate="G$1" pin="PB02(AIN10/SER5:0)"/>
+<wire x1="276.86" y1="200.66" x2="266.7" y2="200.66" width="0.1524" layer="91"/>
+<label x="266.7" y="200.66" size="1.016" layer="95" rot="R180" xref="yes"/>
 </segment>
 </net>
@@
 </segment>
 </net>
-<net name="PB03_A2" class="0">
+<net name="MPU_INT" class="0">
 <segment>
 <pinref part="U1" gate="G$1" pin="PB03(AIN11/SER5:1)"/>
@@
 </segment>
 </net>
+<net name="MPU_INT" class="0">
+<segment>
+<pinref part="U17" gate="G$1" pin="INT"/>
+<wire x1="339.09" y1="220.98" x2="335.28" y2="220.98" width="0.1524" layer="91"/>
+<label x="335.28" y="220.98" size="1.016" layer="95" rot="R180" xref="yes"/>
+</segment>
+</net>

Commit message: maiboard routing completed
Parts:
- added CS, MISO, MOSI, SCK: DNP, Arduino-utility:TPTP-0.8MM
- added FD4, FD5, FD6: DNP, Arduino-utility:FIDUCIAL-1.5MM
Connections:
- net PA16_S1_MOSI: now also MOSI.P$1
- net PA17_S1_SCK: now also SCK.P$1
- net PA19_S1_MISO: now also MISO.P$1
- net PA20_CS: now also CS.P$1
Changed lines of the file:
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@@
 <part name="R27" library="novaXR" deviceset="10K" device="" value="10K"/>
 <part name="J1" library="Molex - 52437-2471" deviceset="MOLEX_52437-2471" device="MOLEX_52437-2471_0_0"/>
+<part name="FD4" library="Arduino-utility" deviceset="FIDUCIAL" device="-1.5MM" value="DNP"/>
+<part name="FD5" library="Arduino-utility" deviceset="FIDUCIAL" device="-1.5MM" value="DNP"/>
+<part name="FD6" library="Arduino-utility" deviceset="FIDUCIAL" device="-1.5MM" value="DNP"/>
+<part name="MISO" library="Arduino-utility" deviceset="TP" device="TP-0.8MM" value="DNP"/>
+<part name="CS" library="Arduino-utility" deviceset="TP" device="TP-0.8MM" value="DNP"/>
+<part name="SCK" library="Arduino-utility" deviceset="TP" device="TP-0.8MM" value="DNP"/>
+<part name="MOSI" library="Arduino-utility" deviceset="TP" device="TP-0.8MM" value="DNP"/>
 </parts>
 <sheets>
@@
 <instance part="J1" gate="G$0" x="317.246" y="12.7" smashed="yes" rot="MR90">
 <attribute name="NAME" x="314.706" y="12.7" size="2.54" layer="95" rot="R90" align="top-left"/>
+</instance>
+<instance part="MISO" gate="G$1" x="375.92" y="216.662" smashed="yes">
+<attribute name="NAME" x="375.92" y="217.678" size="1.778" layer="95" align="bottom-center"/>
+</instance>
+<instance part="CS" gate="G$1" x="381" y="214.122" smashed="yes">
+<attribute name="NAME" x="381" y="215.138" size="1.778" layer="95" align="bottom-center"/>
+</instance>
+<instance part="SCK" gate="G$1" x="381" y="224.282" smashed="yes">
+<attribute name="NAME" x="381" y="225.298" size="1.778" layer="95" align="bottom-center"/>
+</instance>
+<instance part="MOSI" gate="G$1" x="375.92" y="226.822" smashed="yes">
+<attribute name="NAME" x="375.92" y="227.838" size="1.778" layer="95" align="bottom-center"/>
 </instance>
 </instances>
@@
 <segment>
 <pinref part="U1" gate="G$1" pin="PA19(SER1:3+)"/>
-<wire x1="345.44" y1="215.9" x2="350.52" y2="215.9" width="0.1524" layer="91"/>
 <label x="350.52" y="215.9" size="1.27" layer="95" xref="yes"/>
+<wire x1="345.44" y1="215.9" x2="370.84" y2="215.9" width="0.1524" layer="91"/>
+<pinref part="MISO" gate="G$1" pin="P$1"/>
+<wire x1="370.84" y1="215.9" x2="370.84" y2="214.122" width="0.1524" layer="91"/>
+<wire x1="370.84" y1="214.122" x2="375.92" y2="214.122" width="0.1524" layer="91"/>
 </segment>
 <segment>
@@
 <segment>
 <pinref part="U1" gate="G$1" pin="PA17(I2C/SER1:1+)"/>
-<wire x1="345.44" y1="220.98" x2="350.52" y2="220.98" width="0.1524" layer="91"/>
 <label x="350.52" y="220.98" size="1.27" layer="95" xref="yes"/>
+<pinref part="SCK" gate="G$1" pin="P$1"/>
+<wire x1="345.44" y1="220.98" x2="381" y2="220.98" width="0.1524" layer="91"/>
+<wire x1="381" y1="220.98" x2="381" y2="221.742" width="0.1524" layer="91"/>
 </segment>
 <segment>
@@
 <segment>
 <pinref part="U1" gate="G$1" pin="PA16(I2C/SER1:0+)"/>
-<wire x1="345.44" y1="223.52" x2="350.52" y2="223.52" width="0.1524" layer="91"/>
 <label x="350.52" y="223.52" size="1.27" layer="95" xref="yes"/>
+<pinref part="MOSI" gate="G$1" pin="P$1"/>
+<wire x1="345.44" y1="223.52" x2="375.92" y2="223.52" width="0.1524" layer="91"/>
+<wire x1="375.92" y1="223.52" x2="375.92" y2="224.282" width="0.1524" layer="91"/>
 </segment>
 <segment>
@@
 <segment>
 <pinref part="U1" gate="G$1" pin="PA20(SER5:2+)"/>
-<wire x1="345.44" y1="213.36" x2="350.52" y2="213.36" width="0.1524" layer="91"/>
 <label x="350.52" y="213.36" size="1.27" layer="95" xref="yes"/>
+<wire x1="345.44" y1="213.36" x2="368.3" y2="213.36" width="0.1524" layer="91"/>
+<wire x1="368.3" y1="213.36" x2="368.3" y2="210.82" width="0.1524" layer="91"/>
+<pinref part="CS" gate="G$1" pin="P$1"/>
+<wire x1="368.3" y1="210.82" x2="381" y2="210.82" width="0.1524" layer="91"/>
+<wire x1="381" y1="210.82" x2="381" y2="211.582" width="0.1524" layer="91"/>
 </segment>
 </net>
@@
 <attribute name="VALUE" x="231.14" y="210.82" size="1.778" layer="96" font="vector" rot="R270" align="top-center"/>
 </instance>
+<instance part="FD4" gate="G$1" x="34.29" y="5.08" smashed="yes"/>
+<instance part="FD5" gate="G$1" x="40.64" y="5.08" smashed="yes"/>
+<instance part="FD6" gate="G$1" x="46.99" y="5.08" smashed="yes"/>
 </instances>
 <busses>
