File: Fascia_mainBoard/fasciaMainBoard_V0/fasciaMainBoard_V0.brd (EAGLE design)
At the start: 33.6 x 40.6 mm, 114 parts, among them J1 MOLEX_52437-2471MOLEX_52437-2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, J3 -, J8 TC2030-MCP, Q1 BSS138PS,115, U1 ATSAMD21G-A, U17 MPU-6050, U18 LP5912Q3.3DRVRQ1, U3 NINA-W102, U4 ATECC508A-MAHDA-T, U5 MCP73831T-4ADI_OT, U6 LM2664M6_NOPB, U7 TPS72325QDBVRQ1, U8 TLV70025DDCR, U9 LP5912Q3.3DRVRQ1, Y1 32.768Khz

Commit message: first update to project in year 2020
Connections:
- net VBAT_LVL: now also U1.10; no longer U1.47
- net V_BATT: now also U18.4, U9.4
Routing:
- net V_BATT: track 22.2 -> 28.9 mm, vias 1 -> 2
- net VBAT_LVL: track 7.18 -> 5.92 mm
Other:
- board text added: "FACIA_MAINBOARD_V0.1_1/12/20"
- board text removed: "FACIA_MAINBOARD_V0_11/21/19"
Changed lines of the file:
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@@
 <?xml version="1.0" encoding="utf-8"?>
 <!DOCTYPE eagle SYSTEM "eagle.dtd">
-<eagle version="9.5.2">
+<eagle version="9.5.1">
 <drawing>
 <settings>
-<setting alwaysvectorfont="yes"/>
+<setting alwaysvectorfont="no"/>
 <setting verticaltext="up"/>
 </settings>
@@
 <text x="27.2" y="32.5" size="0.6096" layer="26" ratio="20" rot="MR180">MOSI</text>
 <text x="28.3" y="33.9" size="0.6096" layer="26" ratio="20" rot="MR180">CS</text>
-<text x="30.9" y="52.1" size="0.8128" layer="25" ratio="13" distance="61">FACIA_MAINBOARD_V0_11/21/19</text>
+<text x="30.9" y="52.1" size="0.8128" layer="25" ratio="13" distance="61">FACIA_MAINBOARD_V0.1_1/12/20</text>
 </plain>
 <attributes>
@@
 <contactref element="R23" pad="1"/>
 <contactref element="R24" pad="2"/>
-<contactref element="U1" pad="47"/>
 <wire x1="39.753" y1="26.283" x2="38.8045" y2="26.283" width="0.254" layer="1"/>
 <wire x1="38.8045" y1="26.283" x2="38.684" y2="26.4035" width="0.254" layer="1"/>
@@
 <wire x1="40.9" y1="28.5" x2="41.6" y2="28.5" width="0.254" layer="16"/>
 <wire x1="41.6" y1="28.5" x2="41.657" y2="28.443" width="0.254" layer="16"/>
-<wire x1="41.657" y1="28.443" x2="41.657" y2="27.188" width="0.254" layer="16"/>
+<contactref element="U1" pad="10"/>
+<wire x1="41.657" y1="28.443" x2="39.657" y2="33.188" width="0" layer="19" extent="16-16"/>
 </signal>
 <signal name="N$10">
@@
 <wire x1="40" y1="16.225" x2="39.775" y2="16" width="0.4064" layer="16"/>
 <wire x1="40" y1="17" x2="40" y2="16.225" width="0.4064" layer="16"/>
-<wire x1="39.775" y1="16" x2="45.425" y2="16" width="0.4064" layer="16"/>
+<wire x1="39.775" y1="16" x2="40" y2="16" width="0.4064" layer="16"/>
+<wire x1="40" y1="16" x2="45.425" y2="16" width="0.4064" layer="16"/>
 <wire x1="39.6" y1="20.2738" x2="40.4738" y2="20.2738" width="0.254" layer="1"/>
 <wire x1="40.825" y1="20.625" x2="40.825" y2="21.55" width="0.254" layer="1"/>
@@
 <wire x1="38.7" y1="20.6" x2="39.0286" y2="20.2714" width="0.254" layer="1"/>
 <wire x1="39.0286" y1="20.2714" x2="39.6" y2="20.2714" width="0.254" layer="1"/>
-<wire x1="39.753" y1="23.853" x2="38.7" y2="22.8" width="0.254" layer="1"/>
+<wire x1="39.753" y1="23.853" x2="39.3" y2="23.4" width="0.254" layer="1"/>
+<wire x1="39.3" y1="23.4" x2="38.7" y2="22.8" width="0.254" layer="1"/>
 <wire x1="39.6" y1="20.2738" x2="39.6" y2="20.2714" width="0.19" layer="1"/>
+<contactref element="U9" pad="4"/>
+<contactref element="U18" pad="4"/>
+<wire x1="40.825" y1="22.85" x2="39.85" y2="22.85" width="0.254" layer="1"/>
+<wire x1="39.85" y1="22.85" x2="39.3" y2="23.4" width="0.254" layer="1"/>
+<wire x1="36.475" y1="16.05" x2="36.475" y2="15.425" width="0.254" layer="1"/>
+<via x="39.8" y="15.2" extent="1-16" drill="0.25"/>
+<wire x1="39.8" y1="15.2" x2="39.8" y2="15.8" width="0.254" layer="16"/>
+<wire x1="39.8" y1="15.8" x2="40" y2="16" width="0.254" layer="16"/>
+<wire x1="36.475" y1="15.425" x2="36.7" y2="15.2" width="0.254" layer="1"/>
+<wire x1="36.7" y1="15.2" x2="39.8" y2="15.2" width="0.254" layer="1"/>
 </signal>
 <signal name="N$31">
