File: Fascia_physioBoard/fascia_physioBoardV0/Fascia_physioBoardV0.sch (EAGLE design)
At the start: 88 parts, among them CN2 CA0612KRX7R9BB102, CN3 CA0612KRX7R9BB102, CN4 CA0612KRX7R9BB102, CN5 CA0612KRX7R9BB102, CN6 CA0612KRX7R9BB102, J1 MOLEX_52437-2471MOLEX_52437-2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, J2 MOLEX_52437-2471MOLEX_52437-2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, J3 MOLEX_51296-1294MOLEX_51296-1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, U1 ADS1299-X, U10 TPD4E1B06DCKR, U11 TPD4E1B06DCKR, U12 OPA320AIDBVRDBV5-L, U13 ADUM5028, U2 OPA2320AIDGKT_NOVA8-SOIC-L, U3 OPA2320AIDGKT_NOVAL8-SOIC-L, U4 HCNR200-300E, U5 OPA320AIDBVRDBV5-L, U6 TPD4E1B06DCKR, U7 TPD4E1B06DCKR, U8 TPD4E1B06DCKR, U9 TPD4E1B06DCKR

Commit message: fixed issues related to missing traces from pin 1 to the feedback to pin 2
Other:
- note added: "PCB is missing this trace"
Changed lines of the file:
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@@
 <?xml version="1.0" encoding="utf-8"?>
 <!DOCTYPE eagle SYSTEM "eagle.dtd">
-<eagle version="9.5.2">
+<eagle version="9.4.2">
 <drawing>
 <settings>
@@
 <wire x1="327.66" y1="100.24" x2="429.26" y2="100.24" width="0.1524" layer="94"/>
 <text x="198.12" y="53.34" size="2.1844" layer="95">ADUM5028</text>
+<wire x1="177.8" y1="78.74" x2="177.8" y2="63.5" width="0.1524" layer="101"/>
+<wire x1="177.8" y1="63.5" x2="193.04" y2="63.5" width="0.1524" layer="101"/>
+<wire x1="193.04" y1="63.5" x2="193.04" y2="78.74" width="0.1524" layer="101"/>
+<wire x1="193.04" y1="78.74" x2="177.8" y2="78.74" width="0.1524" layer="101"/>
+<text x="175.26" y="60.96" size="1.778" layer="101">PCB is missing this trace</text>
 </plain>
 <instances>
