File: OptoIsolator/SeanOptoIsolatorCircuit.brd (EAGLE design)
At the start: 160 x 100 mm, 10 parts, among them Q1 BROADCOM_HCNR200-300EBROADCOM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, U1 MCP6002-E/SNSOIC8-N_MC-L, U2 MCP6002-E/SNSOIC8-N_MC-L

Commit message: made changes to eda schematic and board files. fixing the issues preventing the V0 to work correctly
Connections:
- removed net N$6: Q1.5, U2.3
- net GND-ISO: now also Q1.5, U2.3
Changed lines of the file:
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@@
 <wire x1="17.145" y1="21.3614" x2="29.21" y2="14.685" width="0" layer="19" extent="1-1"/>
 </signal>
-<signal name="N$6">
+<signal name="GND-ISO">
+<contactref element="U2" pad="4"/>
 <contactref element="Q1" pad="5"/>
 <contactref element="U2" pad="3"/>
 <wire x1="15.875" y1="21.3614" x2="26.67" y2="14.685" width="0" layer="19" extent="1-1"/>
-</signal>
-<signal name="GND-ISO">
-<contactref element="U2" pad="4"/>
+<wire x1="14.605" y1="21.3614" x2="15.875" y2="21.3614" width="0" layer="19" extent="1-1"/>
 </signal>
 <signal name="VCC-ISO">
