File: Fascia_faceInterface/fascia_faceInterfaceV0.brd (EAGLE design)
At the start: 200 x 112.8 mm, 20 parts, among them J1 MOLEX_52437-247_FLEX, J2 SM04B-SRSS-TB(LF)(SN)

Commit message: flexible boards files submitted for fabrication
Parts:
- moved J1 3.61 mm to (52.8, 120.3)
Routing:
- net AGND: track 0.00 -> 49.7 mm, vias 14 -> 15
- net S0_I2C_SDA: track 40.0 -> 88.6 mm
- net S0_I2C_SCL: track 39.7 -> 88.2 mm
- net 1P: track 40.2 -> 88.6 mm
- net 2P: track 53.1 -> 101.2 mm
- net 3P: track 196.8 -> 244.8 mm
- net 3N: track 213.7 -> 261.4 mm
- net 4P: track 45.3 -> 92.9 mm
- net 4N: track 64.0 -> 111.2 mm
- net DVDD: track 46.7 -> 93.9 mm
- net 5P: track 132.5 -> 179.6 mm
- net 5N: track 132.9 -> 179.9 mm
- net 6P: track 64.4 -> 111.1 mm
- net 6N: track 45.4 -> 92.0 mm
- net 7P: track 80.3 -> 126.8 mm
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- removed copper zone on layer 1, net AGND
Other:
- board size 200 x 112.8 mm -> 200 x 123.7 mm
- board text added: "fascia-faceInterfaceV0-Bernal-031020"
- board text added: "stiffener BOT"
- board text removed: "novaXR-faceInterfaceV1-Bernal-082919"
- board text removed: "stiffener TOP"
