File: Fascia_mainBoard/fasciaMainBoard_V0.1/fasciaMainBoard_V0.1.brd (EAGLE design)
At the start: 33.6 x 40.6 mm, 114 parts, among them J1 MOLEX_52437-2471MOLEX_52437-2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, J3 -, J8 TC2030-MCP, Q1 BSS138PS,115, U1 ATSAMD21G-A, U17 MPU-6050, U18 LP5912Q3.3DRVRQ1, U3 NINA-W102, U4 ATECC508A-MAHDA-T, U5 MCP73831T-4ADI_OT, U6 LM2664M6_NOPB, U7 TPS72325QDBVRQ1, U8 TLV70025DDCR, U9 LP5912Q3.3DRVRQ1, Y1 32.768Khz

Commit message: changes to the fascia boards
Connections:
- removed net ADS_CLK: J1.22
- net PB11_CLKSEL: now also J1.22
Routing:
- net PB11_CLKSEL: track 0.00 -> 19.6 mm, vias 0 -> 2
- net RESET#: track 19.6 -> 20.5 mm
- net PB10_DRDY: track 18.4 -> 19.1 mm

Commit message: flexible boards files submitted for fabrication
Parts:
- removed C34, C35: 0.1uF, novaXR:0402-TIGHT
- removed C36: 0.01uF, novaXR:0402-TIGHT
- removed C37: 2.2nF, novaXR:0402-TIGHT
- removed U17: MPU-6050, SamacSys_Parts:MPU6050
Connections:
- removed net N$37: C35.2, U17.10
- removed net N$39: C37.2, U17.20
- net GND: no longer C34.1, C35.1, C36.1, C37.1, U17.1, U17.11, U17.18, U17.9
- net MPU_INT: no longer U17.12
- net S0_I2C_SCL: no longer U17.23
- net S0_I2C_SDA: no longer U17.24
- net VCC: no longer C34.2, C36.2, U17.13, U17.8
Routing:
- net GND: track 139.1 -> 130.3 mm, vias 33 -> 30
- net VCC: track 57.9 -> 55.2 mm, vias 15 -> 13
- net N$37: track 1.70 -> 0.00 mm
- net S0_I2C_SCL: track 23.8 -> 22.7 mm
- net N$39: track 1.03 -> 0.00 mm
- net S0_I2C_SDA: track 20.1 -> 19.2 mm

Commit message: update to board files for manufacturing
Parts:
- added C15, C35: 0.1uF, SparkFun-Capacitors:0402
- added C34: 10NF0402-5%, SparkFun-Capacitors:0402
- added U17: MPU6050, invensense:QFN50P400X400X95-25T265X275N
Connections:
- new net N$14: C35.1, U17.13
- new net N$5: C15.1, U17.10
- net GND: now also C15.2, C34.2, C35.2, U17.1, U17.18, U17.25, U17.9
- net MPU_INT: now also U17.12
- net S0_I2C_SCL: now also U17.23
- net S0_I2C_SDA: now also U17.24
- net VCC: now also C34.1, U17.8
Routing:
- net GND: track 130.3 -> 143.8 mm, vias 30 -> 33
- net MPU_INT: track 16.7 -> 23.2 mm
- net VCC: track 55.2 -> 59.7 mm
- net S0_I2C_SDA: track 19.2 -> 23.2 mm
- net S0_I2C_SCL: track 22.7 -> 25.3 mm
- net N$14: track 0.00 -> 1.65 mm
- net N$5: track 0.00 -> 1.64 mm
- added copper zone on layer 16, net GND
Other:
- board text added: "FACIA_MAINBOARD_V0.1_3/12/20"
- board text removed: "FACIA_MAINBOARD_V0.1_1/12/20"
