File: Fascia_mainBoard/fasciaMainBoard_V0.1/fasciaMainBoard_V0.1.sch (EAGLE design)
At the start: 114 parts, among them J1 MOLEX_52437-2471MOLEX_52437-2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, J3 -, J8 TC2030-MCP, Q1 BSS138PS,115, U1 ATSAMD21G-A, U17 MPU-6050, U18 LP5912Q3.3DRVRQ1, U3 NINA-W102, U4 ATECC508A-MAHDA-T, U5 MCP73831T-4ADI_OT, U6 LM2664M6_NOPB, U7 TPS72325QDBVRQ1, U8 TLV70025DDCR, U9 LP5912Q3.3DRVRQ1, Y1 32.768Khz

Commit message: first update to project in year 2020
Connections:
- removed net PA07_DRDY: J1.18, U1.PA07(AIN7/SER0:3/TC1:1)
- new net PB10_DRDY: J1.18, U1.PB10(SER4:2+)
- net VBAT_LVL: now also U1.PA03(AIN1/REFA); no longer U1.PB02(AIN10/SER5:0)
- net V_BATT: now also U18.EN, U9.EN
Changed lines of the file:
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@@
-</segment>
-</net>
-<net name="VBAT_LVL" class="0">
-<segment>
-<pinref part="U1" gate="G$1" pin="PB02(AIN10/SER5:0)"/>
-<wire x1="276.86" y1="200.66" x2="266.7" y2="200.66" width="0.1524" layer="91"/>
-<label x="266.7" y="200.66" size="1.016" layer="95" rot="R180" xref="yes"/>
 </segment>
 </net>
@@
 </segment>
 </net>
-<net name="PA07_DRDY" class="0">
-<segment>
-<pinref part="U1" gate="G$1" pin="PA07(AIN7/SER0:3/TC1:1)"/>
-<wire x1="276.86" y1="203.2" x2="266.7" y2="203.2" width="0.1524" layer="91"/>
-<label x="266.7" y="203.2" size="1.016" layer="95" rot="R180" xref="yes"/>
+<net name="PB10_DRDY" class="0">
+<segment>
+<pinref part="U1" gate="G$1" pin="PB10(SER4:2+)"/>
+<wire x1="345.44" y1="185.42" x2="353.06" y2="185.42" width="0.1524" layer="91"/>
+<label x="353.06" y="185.42" size="0.8128" layer="95" xref="yes"/>
 </segment>
 <segment>
@@
 <wire x1="297.18" y1="58.42" x2="287.02" y2="58.42" width="0.1524" layer="91"/>
 <wire x1="299.5676" y1="58.42" x2="302.006" y2="58.42" width="0.1524" layer="91"/>
+</segment>
+</net>
+<net name="VBAT_LVL" class="0">
+<segment>
+<pinref part="U1" gate="G$1" pin="PA03(AIN1/REFA)"/>
+<wire x1="276.86" y1="213.36" x2="274.32" y2="213.36" width="0.1524" layer="91"/>
+<label x="274.32" y="213.36" size="0.8128" layer="95" rot="R180" xref="yes"/>
 </segment>
 </net>
@@
 </instance>
 <instance part="U18" gate="G$1" x="233.68" y="223.52" smashed="yes">
-<attribute name="NAME" x="249.2756" y="232.6386" size="2.0828" layer="95" ratio="6" rot="SR0"/>
-<attribute name="VALUE" x="248.6406" y="230.0986" size="2.0828" layer="96" ratio="6" rot="SR0"/>
+<attribute name="NAME" x="239.1156" y="232.6386" size="2.0828" layer="95" ratio="6" rot="SR0"/>
+<attribute name="VALUE" x="241.0206" y="230.0986" size="2.0828" layer="96" ratio="6" rot="SR0"/>
 </instance>
 <instance part="C18" gate="A" x="223.52" y="213.36" smashed="yes" rot="R90">
@@
 <segment>
 <pinref part="U18" gate="G$1" pin="PAD"/>
-<wire x1="271.78" y1="223.52" x2="274.32" y2="223.52" width="0.1524" layer="91"/>
-<label x="274.32" y="223.52" size="1.778" layer="95" rot="R90" xref="yes"/>
+<wire x1="271.78" y1="223.52" x2="279.4" y2="223.52" width="0.1524" layer="91"/>
+<label x="279.4" y="223.52" size="1.778" layer="95" rot="R90" xref="yes"/>
 </segment>
 </net>
@@
 <junction x="284.48" y="220.98"/>
 </segment>
-</net>
+<segment>
+<pinref part="U9" gate="G$1" pin="EN"/>
+<wire x1="271.78" y1="248.92" x2="271.78" y2="243.84" width="0.1524" layer="91"/>
+<label x="271.78" y="243.84" size="0.8128" layer="95" rot="R270" xref="yes"/>
+</segment>
+<segment>
+<pinref part="U18" gate="G$1" pin="EN"/>
+<wire x1="271.78" y1="215.9" x2="271.78" y2="210.82" width="0.1524" layer="91"/>
+<label x="271.78" y="210.82" size="0.8128" layer="95" rot="R270" xref="yes"/>
+</segment>
+</net>

Commit message: changes to the fascia boards
Connections:
- removed net ADS_CLK: J1.22
- net PB11_CLKSEL: now also J1.22
Changed lines of the file:
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@@
 <label x="353.06" y="182.88" size="1.016" layer="95" xref="yes"/>
+</segment>
+<segment>
+<label x="287.02" y="68.58" size="1.016" layer="95" rot="R180" xref="yes"/>
+<wire x1="299.5676" y1="68.58" x2="297.18" y2="68.58" width="0.1524" layer="91"/>
+<pinref part="J1" gate="G$0" pin="22"/>
+<wire x1="297.18" y1="68.58" x2="287.02" y2="68.58" width="0.1524" layer="91"/>
+<wire x1="299.5676" y1="68.58" x2="302.006" y2="68.58" width="0.1524" layer="91"/>
 </segment>
 </net>
@@
 </segment>
 </net>
-<net name="ADS_CLK" class="0">
-<segment>
-<label x="287.02" y="68.58" size="1.016" layer="95" rot="R180" xref="yes"/>
-<wire x1="299.5676" y1="68.58" x2="297.18" y2="68.58" width="0.1524" layer="91"/>
-<pinref part="J1" gate="G$0" pin="22"/>
-<wire x1="297.18" y1="68.58" x2="287.02" y2="68.58" width="0.1524" layer="91"/>
-<wire x1="299.5676" y1="68.58" x2="302.006" y2="68.58" width="0.1524" layer="91"/>
-</segment>
-</net>

Commit message: flexible boards files submitted for fabrication
Parts:
- removed C34, C35: 0.1uF, novaXR:0.1UF-0402T-16V-10%
- removed C36: 0.01uF, novaXR:0.01UF-0402T-16V-10%
- removed C37: 2.2nF, novaXR:2.2NF-0402T-16V-10%
- removed U17: MPU-6050, SamacSys_Parts:MPU-6050
Connections:
- removed net N$37: C35.2, U17.REGOUT
- removed net N$39: C37.2, U17.CPOUT
- net GND: no longer C34.1, C35.1, C36.1, C37.1, U17.AD0, U17.CLKIN, U17.FSYNC, U17.GND
- net MPU_INT: no longer U17.INT
- net S0_I2C_SCL: no longer U17.SCL
- net S0_I2C_SDA: no longer U17.SDA
- net VCC: no longer C34.2, C36.2, U17.VDD, U17.VLOGIC
Changed lines of the file:
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@@
 <part name="GND38" library="SparkFun-PowerSymbols" library_urn="urn:adsk.eagle:library:530" deviceset="GND" device=""/>
 <part name="C33" library="novaXR" deviceset="0.1UF" device="-0402T-16V-10%" value="0.1uF"/>
-<part name="U17" library="SamacSys_Parts" deviceset="MPU-6050" device=""/>
-<part name="C34" library="novaXR" deviceset="0.1UF" device="-0402T-16V-10%" value="0.1uF"/>
-<part name="GND39" library="SparkFun-PowerSymbols" library_urn="urn:adsk.eagle:library:530" deviceset="GND" device=""/>
-<part name="GND40" library="SparkFun-PowerSymbols" library_urn="urn:adsk.eagle:library:530" deviceset="GND" device=""/>
-<part name="C35" library="novaXR" deviceset="0.1UF" device="-0402T-16V-10%" value="0.1uF"/>
-<part name="C36" library="novaXR" deviceset="0.01UF" device="-0402T-16V-10%" value="0.01uF"/>
-<part name="C37" library="novaXR" deviceset="2.2NF" device="-0402T-16V-10%" value="2.2nF"/>
 <part name="J3" library="Arduino-connectors" deviceset="USB-MICRO" device="" value="-"/>
 <part name="D2" library="Arduino-diodes" deviceset="PRTR5V0U2X,215" device="" value="PRTR5V"/>
@@
 <part name="U$32" library="supply1" deviceset="AVSS" device=""/>
 <part name="U$33" library="supply1" deviceset="AVDD" device=""/>
-<part name="U$35" library="SparkFun-PowerSymbols" deviceset="VCC" device=""/>
 <part name="U$36" library="SparkFun-PowerSymbols" deviceset="VCC" device=""/>
 <part name="U$37" library="SparkFun-PowerSymbols" deviceset="VCC" device=""/>
@@
 <part name="GND8" library="SparkFun-PowerSymbols" library_urn="urn:adsk.eagle:library:530" deviceset="GND" device=""/>
 <part name="SUPPLY3" library="SparkFun-PowerSymbols" deviceset="VCC" device=""/>
-<part name="U$6" library="SparkFun-PowerSymbols" deviceset="VCC" device=""/>
 <part name="U$25" library="supply1" deviceset="DVDD" device=""/>
 <part name="U9" library="Lp5912Q3.3DRV" deviceset="LP5912Q3.3DRVRQ1" device=""/>
@@
 <attribute name="VALUE" x="78.486" y="177.419" size="1.778" layer="96" font="vector" rot="R180"/>
 </instance>
-<instance part="U17" gate="G$1" x="339.09" y="248.92" smashed="yes">
-<attribute name="NAME" x="344.17" y="255.27" size="1.778" layer="95" align="center-left"/>
-<attribute name="VALUE" x="344.17" y="252.73" size="1.778" layer="96" align="center-left"/>
-</instance>
-<instance part="C34" gate="G$1" x="317.5" y="210.82" smashed="yes" rot="R180">
-<attribute name="NAME" x="316.23" y="208.28" size="1.778" layer="95" font="vector" rot="R180"/>
-<attribute name="VALUE" x="315.976" y="212.979" size="1.778" layer="96" font="vector" rot="R180"/>
-</instance>
-<instance part="GND39" gate="1" x="317.5" y="200.66" smashed="yes">
-<attribute name="VALUE" x="317.5" y="199.136" size="1.778" layer="96" align="top-center"/>
-</instance>
-<instance part="GND40" gate="1" x="382.27" y="203.2" smashed="yes">
-<attribute name="VALUE" x="382.27" y="201.676" size="1.778" layer="96" align="top-center"/>
-</instance>
-<instance part="C35" gate="G$1" x="325.12" y="210.82" smashed="yes" rot="R180">
-<attribute name="NAME" x="323.85" y="208.28" size="1.778" layer="95" font="vector" rot="R180"/>
-<attribute name="VALUE" x="323.596" y="212.979" size="1.778" layer="96" font="vector" rot="R180"/>
-</instance>
-<instance part="C36" gate="G$1" x="334.01" y="210.82" smashed="yes" rot="R180">
-<attribute name="NAME" x="332.74" y="208.28" size="1.778" layer="95" font="vector" rot="R180"/>
-<attribute name="VALUE" x="332.486" y="212.979" size="1.778" layer="96" font="vector" rot="R180"/>
-</instance>
-<instance part="C37" gate="G$1" x="379.73" y="218.44" smashed="yes" rot="R180">
-<attribute name="NAME" x="378.46" y="215.9" size="1.778" layer="95" font="vector" rot="R180"/>
-<attribute name="VALUE" x="378.206" y="220.599" size="1.778" layer="96" font="vector" rot="R180"/>
-</instance>
 <instance part="J3" gate="G$1" x="17.78" y="226.06" smashed="yes">
 <attribute name="NAME" x="20.32" y="239.522" size="1.778" layer="95" align="bottom-center"/>
@@
 <attribute name="VALUE" x="274.32" y="185.928" size="1.778" layer="96"/>
 </instance>
-<instance part="U$35" gate="G$1" x="317.5" y="220.472" smashed="yes">
-<attribute name="VALUE" x="321.056" y="226.06" size="1.778" layer="96" rot="R180"/>
-</instance>
 <instance part="J6" gate="G$1" x="171.45" y="262.89" smashed="yes" rot="R90">
 <attribute name="NAME" x="165.735" y="256.54" size="1.778" layer="95" rot="R90"/>
@@
 <instance part="SUPPLY3" gate="G$1" x="223.52" y="226.06" smashed="yes">
 <attribute name="VALUE" x="223.52" y="228.854" size="1.778" layer="96" align="bottom-center"/>
-</instance>
-<instance part="U$6" gate="G$1" x="317.5" y="235.712" smashed="yes">
-<attribute name="VALUE" x="321.056" y="241.3" size="1.778" layer="96" rot="R180"/>
 </instance>
 <instance part="U$25" gate="G$1" x="223.52" y="259.08" smashed="yes">
@@
 </segment>
 <segment>
-<pinref part="C34" gate="G$1" pin="1"/>
-<pinref part="GND39" gate="1" pin="GND"/>
-<wire x1="317.5" y1="205.74" x2="317.5" y2="203.2" width="0.1524" layer="91"/>
-<pinref part="C37" gate="G$1" pin="1"/>
-<wire x1="379.73" y1="213.36" x2="379.73" y2="205.74" width="0.1524" layer="91"/>
-<wire x1="379.73" y1="205.74" x2="334.01" y2="205.74" width="0.1524" layer="91"/>
-<pinref part="C35" gate="G$1" pin="1"/>
-<junction x="325.12" y="205.74"/>
-<wire x1="334.01" y1="205.74" x2="325.12" y2="205.74" width="0.1524" layer="91"/>
-<wire x1="325.12" y1="205.74" x2="317.5" y2="205.74" width="0.1524" layer="91"/>
-<pinref part="C36" gate="G$1" pin="1"/>
-<junction x="334.01" y="205.74"/>
-</segment>
-<segment>
-<pinref part="U17" gate="G$1" pin="GND"/>
-<wire x1="372.11" y1="238.76" x2="382.27" y2="238.76" width="0.1524" layer="91"/>
-<wire x1="382.27" y1="238.76" x2="382.27" y2="205.74" width="0.1524" layer="91"/>
-<pinref part="GND40" gate="1" pin="GND"/>
-</segment>
-<segment>
-<pinref part="U17" gate="G$1" pin="CLKIN"/>
-<wire x1="339.09" y1="248.92" x2="335.28" y2="248.92" width="0.1524" layer="91"/>
-<label x="335.28" y="248.92" size="1.778" layer="95" rot="R180" xref="yes"/>
-</segment>
-<segment>
-<wire x1="339.09" y1="223.52" x2="336.55" y2="223.52" width="0.1524" layer="91"/>
-<label x="336.55" y="223.52" size="1.778" layer="95" rot="R180" xref="yes"/>
-<pinref part="U17" gate="G$1" pin="FSYNC"/>
-</segment>
-<segment>
 <pinref part="J3" gate="G$1" pin="5"/>
 <wire x1="25.4" y1="220.98" x2="25.4" y2="218.44" width="0.1524" layer="91"/>
@@
 <pinref part="GND48" gate="1" pin="GND"/>
 <wire x1="25.4" y1="242.57" x2="26.67" y2="242.57" width="0.1524" layer="91"/>
-</segment>
-<segment>
-<wire x1="339.09" y1="228.6" x2="336.55" y2="228.6" width="0.1524" layer="91"/>
-<label x="336.55" y="228.6" size="1.778" layer="95" rot="R180" xref="yes"/>
-<pinref part="U17" gate="G$1" pin="AD0"/>
 </segment>
 <segment>
@@
 <junction x="80.01" y="180.34"/>
 <label x="80.01" y="195.58" size="1.778" layer="95" xref="yes"/>
-</segment>
-</net>
-<net name="N$37" class="0">
-<segment>
-<pinref part="C35" gate="G$1" pin="2"/>
-<pinref part="U17" gate="G$1" pin="REGOUT"/>
-<wire x1="325.12" y1="213.36" x2="325.12" y2="226.06" width="0.1524" layer="91"/>
-<wire x1="325.12" y1="226.06" x2="339.09" y2="226.06" width="0.1524" layer="91"/>
-</segment>
-</net>
-<net name="N$39" class="0">
-<segment>
-<pinref part="C37" gate="G$1" pin="2"/>
-<wire x1="379.73" y1="220.98" x2="379.73" y2="233.68" width="0.1524" layer="91"/>
-<pinref part="U17" gate="G$1" pin="CPOUT"/>
-<wire x1="379.73" y1="233.68" x2="372.11" y2="233.68" width="0.1524" layer="91"/>
-</segment>
-</net>
-<net name="S0_I2C_SCL" class="0">
-<segment>
-<pinref part="U17" gate="G$1" pin="SCL"/>
-<wire x1="372.11" y1="226.06" x2="383.54" y2="226.06" width="0.1524" layer="91"/>
-<label x="383.54" y="226.06" size="1.778" layer="95" xref="yes"/>
-</segment>
-</net>
-<net name="S0_I2C_SDA" class="0">
-<segment>
-<pinref part="U17" gate="G$1" pin="SDA"/>
-<wire x1="372.11" y1="223.52" x2="400.05" y2="223.52" width="0.1524" layer="91"/>
-<label x="400.05" y="223.52" size="1.778" layer="95" xref="yes"/>
 </segment>
 </net>
@@
 <net name="VCC" class="0">
 <segment>
-<pinref part="C34" gate="G$1" pin="2"/>
-<wire x1="317.5" y1="213.36" x2="317.5" y2="220.472" width="0.1524" layer="91"/>
-<wire x1="317.5" y1="220.472" x2="317.5" y2="220.98" width="0.1524" layer="91"/>
-<wire x1="340.36" y1="218.44" x2="339.09" y2="218.44" width="0.1524" layer="91"/>
-<junction x="317.5" y="213.36"/>
-<pinref part="U17" gate="G$1" pin="VDD"/>
-<wire x1="339.09" y1="218.44" x2="317.5" y2="218.44" width="0.1524" layer="91"/>
-<wire x1="317.5" y1="218.44" x2="317.5" y2="213.36" width="0.1524" layer="91"/>
-<junction x="339.09" y="218.44"/>
-<pinref part="U$35" gate="G$1" pin="VCC"/>
-<junction x="317.5" y="220.472"/>
-<wire x1="317.5" y1="220.472" x2="317.5" y2="220.98" width="0.1524" layer="91"/>
-</segment>
-<segment>
-<pinref part="C36" gate="G$1" pin="2"/>
-<wire x1="334.01" y1="213.36" x2="334.01" y2="231.14" width="0.1524" layer="91"/>
-<pinref part="U17" gate="G$1" pin="VLOGIC"/>
-<wire x1="334.01" y1="231.14" x2="335.28" y2="231.14" width="0.1524" layer="91"/>
-<pinref part="U$6" gate="G$1" pin="VCC"/>
-<wire x1="335.28" y1="231.14" x2="339.09" y2="231.14" width="0.1524" layer="91"/>
-<wire x1="334.01" y1="231.14" x2="317.5" y2="231.14" width="0.1524" layer="91"/>
-<wire x1="317.5" y1="231.14" x2="317.5" y2="235.712" width="0.1524" layer="91"/>
-</segment>
-<segment>
 <pinref part="U18" gate="G$1" pin="OUT"/>
 <pinref part="C18" gate="A" pin="2"/>
@@
 </segment>
 </net>
-<net name="MPU_INT" class="0">
-<segment>
-<pinref part="U17" gate="G$1" pin="INT"/>
-<wire x1="339.09" y1="220.98" x2="335.28" y2="220.98" width="0.1524" layer="91"/>
-<label x="335.28" y="220.98" size="1.016" layer="95" rot="R180" xref="yes"/>
-</segment>
-</net>

Commit message: update to board files for manufacturing
Parts:
- added C15, C35: 0.1uF, SparkFun-Capacitors:0.1UF-0402-16V-10%
- added C34: 10NF0402-5%, SparkFun-Capacitors:10NF0402-5%
- added U17: MPU6050, invensense:MPU6050
Connections:
- new net N$14: C35.1, U17G$1.VDD
- new net N$5: C15.1, U17G$1.REGOUT
- net GND: now also C15.2, C34.2, C35.2, U17G$1.AD0, U17G$1.CLKIN, U17G$1.GND, U17G$1.GND@1
- net MPU_INT: now also U17G$1.INT
- net S0_I2C_SCL: now also U17G$1.SCL
- net S0_I2C_SDA: now also U17G$1.SDA
- net VCC: now also C34.1, U17G$1.VLOGIC
