File: Fascia_physioBoard/fascia_physioBoardV0.1/Fascia_physioBoardV0.1.brd (EAGLE design)
At the start: 37.3 x 39.1 mm, 86 parts, among them CN2 CA0612KRX7R9BB102, CN3 CA0612KRX7R9BB102, CN4 CA0612KRX7R9BB102, CN5 CA0612KRX7R9BB102, CN6 CA0612KRX7R9BB102, J1 MOLEX_52437-2471MOLEX_52437-2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, J2 MOLEX_52437-2471MOLEX_52437-2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, J3 MOLEX_51296-1294MOLEX_51296-1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, U1 ADS1299-X, U10 TPD4E1B06DCKR, U11 TPD4E1B06DCKR, U12 OPA320AIDBVRDBV5-L, U13 ADUM5028, U2 OPA2320AIDGKT_NOVA8-SOIC-L, U3 OPA2320AIDGKT_NOVAL8-SOIC-L, U4 HCNR200-300E, U5 OPA320AIDBVRDBV5-L, U6 TPD4E1B06DCKR, U7 TPD4E1B06DCKR, U8 TPD4E1B06DCKR, U9 TPD4E1B06DCKR

Commit message: changed values used on the board to be reflected on the schematic
Parts:
- R18: value 110K -> 140K
- R7: value 10K -> 20K
- R9: value 875K -> 866K
Changed lines of the file:
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@@
 <?xml version="1.0" encoding="utf-8"?>
 <!DOCTYPE eagle SYSTEM "eagle.dtd">
-<eagle version="9.4.2">
+<eagle version="9.6.0">
 <drawing>
 <settings>
@@
 <layer number="14" name="Route14" color="22" fill="1" visible="no" active="no"/>
 <layer number="15" name="Route15" color="23" fill="1" visible="no" active="yes"/>
-<layer number="16" name="Bottom" color="1" fill="1" visible="yes" active="yes"/>
+<layer number="16" name="Bottom" color="1" fill="1" visible="no" active="yes"/>
 <layer number="17" name="Pads" color="2" fill="1" visible="yes" active="yes"/>
 <layer number="18" name="Vias" color="2" fill="1" visible="yes" active="yes"/>
 <layer number="19" name="Unrouted" color="13" fill="1" visible="yes" active="yes"/>
 <layer number="20" name="Dimension" color="21" fill="1" visible="yes" active="yes"/>
-<layer number="21" name="tPlace" color="7" fill="1" visible="no" active="yes"/>
-<layer number="22" name="bPlace" color="7" fill="1" visible="yes" active="yes"/>
-<layer number="23" name="tOrigins" color="15" fill="1" visible="no" active="yes"/>
-<layer number="24" name="bOrigins" color="15" fill="1" visible="yes" active="yes"/>
+<layer number="21" name="tPlace" color="7" fill="1" visible="yes" active="yes"/>
+<layer number="22" name="bPlace" color="7" fill="1" visible="no" active="yes"/>
+<layer number="23" name="tOrigins" color="15" fill="1" visible="yes" active="yes"/>
+<layer number="24" name="bOrigins" color="15" fill="1" visible="no" active="yes"/>
 <layer number="25" name="tNames" color="7" fill="1" visible="yes" active="yes"/>
-<layer number="26" name="bNames" color="7" fill="1" visible="yes" active="yes"/>
+<layer number="26" name="bNames" color="7" fill="1" visible="no" active="yes"/>
 <layer number="27" name="tValues" color="7" fill="1" visible="no" active="yes"/>
 <layer number="28" name="bValues" color="7" fill="1" visible="no" active="yes"/>
@@
 <layer number="37" name="tTest" color="7" fill="1" visible="no" active="yes"/>
 <layer number="38" name="bTest" color="7" fill="1" visible="no" active="yes"/>
-<layer number="39" name="tKeepout" color="4" fill="11" visible="no" active="yes"/>
-<layer number="40" name="bKeepout" color="1" fill="11" visible="yes" active="yes"/>
-<layer number="41" name="tRestrict" color="4" fill="10" visible="no" active="yes"/>
-<layer number="42" name="bRestrict" color="1" fill="10" visible="yes" active="yes"/>
+<layer number="39" name="tKeepout" color="4" fill="11" visible="yes" active="yes"/>
+<layer number="40" name="bKeepout" color="1" fill="11" visible="no" active="yes"/>
+<layer number="41" name="tRestrict" color="4" fill="10" visible="yes" active="yes"/>
+<layer number="42" name="bRestrict" color="1" fill="10" visible="no" active="yes"/>
 <layer number="43" name="vRestrict" color="2" fill="10" visible="no" active="yes"/>
 <layer number="44" name="Drills" color="7" fill="1" visible="no" active="yes"/>
@@
 <layer number="50" name="dxf" color="7" fill="1" visible="no" active="no"/>
 <layer number="51" name="tDocu" color="7" fill="1" visible="yes" active="yes"/>
-<layer number="52" name="bDocu" color="7" fill="1" visible="yes" active="yes"/>
+<layer number="52" name="bDocu" color="7" fill="1" visible="no" active="yes"/>
 <layer number="53" name="tGND_GNDA" color="7" fill="9" visible="no" active="no"/>
 <layer number="54" name="bGND_GNDA" color="1" fill="9" visible="no" active="no"/>
@@
 </layers>
 <board>
-<fusionsync huburn="a.cGVyc29uYWw6dWUyOWVjN2Ji" projecturn="a.cGVyc29uYWw6dWUyOWVjN2JiIzIwMTQwOTMwMzkxMDg3Ng" f3durn="urn:adsk.wipprod:dm.lineage:D7K6kwDeRD-gceEODQpGvg" pcbguid="de4ec628-bd80-46e9-b935-15577d277fac" lastpulledtime="" lastsyncedchangeguid="3500d560-1b9a-7ecd-289c-2de5f38b5079"/>
+<fusionsync huburn="a.cGVyc29uYWw6dWUyOWVjN2Ji" projecturn="a.cGVyc29uYWw6dWUyOWVjN2JiIzIwMTQwOTMwMzkxMDg3Ng" f3durn="urn:adsk.wipprod:dm.lineage:D7K6kwDeRD-gceEODQpGvg" pcbguid="de4ec628-bd80-46e9-b935-15577d277fac" lastpulledtime="" lastsyncedchangeguid="3500d560-1b9a-7ecd-289c-2de5f38b5079" latestrevisionid="" lastsyncedrevisionid="" lastboardhashguid="" lastpushedtime="" linktopcb3d="%12"/>
 <plain>
 <text x="23" y="20.6" size="0.4064" layer="26" ratio="10" rot="MR0">GND_ISO</text>
@@
 <attribute name="VALUE" value="47uF" x="16.088" y="18.65" size="0.6096" layer="28" font="vector" ratio="20" rot="MR90" align="top-center"/>
 </element>
-<element name="R9" library="novaXR" package="0402-TIGHT" value="875K" x="17.15" y="20.85" smashed="yes" rot="MR0">
+<element name="R9" library="novaXR" package="0402-TIGHT" value="866K" x="17.15" y="20.85" smashed="yes" rot="MR0">
 <attribute name="NAME" x="18.55" y="20.312" size="0.6096" layer="26" font="vector" ratio="20" rot="MR0" align="bottom-center"/>
 <attribute name="VALUE" value="875K" x="17.15" y="20.088" size="0.6096" layer="28" font="vector" ratio="20" rot="MR0" align="top-center"/>
@@
 <attribute name="VALUE" x="2.268" y="32.17" size="0.6096" layer="27" font="vector" ratio="20" rot="R270"/>
 </element>
-<element name="R7" library="novaXR" package="0402-TIGHT" value="10K" x="18.3" y="14.3" smashed="yes" rot="MR90">
-<attribute name="NAME" x="18.862" y="14.3" size="0.6096" layer="26" font="vector" ratio="20" rot="MR90" align="bottom-center"/>
+<element name="R7" library="novaXR" package="0402-TIGHT" value="20K" x="18.3" y="14.3" smashed="yes" rot="MR90">
+<attribute name="NAME" x="18.062" y="16" size="0.6096" layer="26" font="vector" ratio="20" rot="MR90" align="bottom-center"/>
 <attribute name="VALUE" x="17.738" y="14.3" size="0.6096" layer="28" font="vector" ratio="20" rot="MR90" align="top-center"/>
 </element>
-<element name="R18" library="novaXR" package="0402-TIGHT" value="110K" x="17.4" y="14.3" smashed="yes" rot="MR270">
+<element name="R18" library="novaXR" package="0402-TIGHT" value="140K" x="17.4" y="14.3" smashed="yes" rot="MR270">
 <attribute name="NAME" x="17.7" y="13.138" size="0.6096" layer="26" font="vector" ratio="20" rot="MR180" align="bottom-center"/>
 <attribute name="VALUE" x="17.962" y="14.3" size="0.6096" layer="28" font="vector" ratio="20" rot="MR270" align="top-center"/>
